File: pcb_files/mouse/mouse_v2.kicad_pcb (KiCad board)
At the start: 2 copper layers, 84.9 x 94.9 mm, 67 parts, among them J1 Conn_01x06_Female, J2 Conn_01x02_Female, J3 Conn_01x02_Male, J4 I2C_Conn, M1 Motor_DC, M2 Motor_DC, Q0 Q_Photo_NPN, Q1 Q_Photo_NPN, Q2 Q_Photo_NPN, Q3 Q_Photo_NPN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

Commit message: V1.2
Parts:
- removed J4: I2C_Conn, Connector_PinSocket_2.54mm:PinSocket_1x02_P2.54mm_Vertical
- added J5: USB_C_Receptacle_USB2.0, Connector_USB:USB_C_Receptacle_GCT_USB4085, F.Cu at (197.3, 112.9)
- added MH3: M3, MountingHole:MountingHole_2.2mm_M2, F.Cu at (181.2, 99.4)
- added MH4: M3, MountingHole:MountingHole_2.2mm_M2, F.Cu at (139.3, 99.4)
- C4: footprint Capacitor_SMD:C_1210_3225Metric_Pad1.42x2.65mm_HandSolder -> Capacitor_SMD:C_1210_3225Metric_Pad1.33x2.70mm_HandSolder
- U1: footprint teensy:Teensy40 -> MCU_RaspberryPi_and_Boards:Teensy40
- U4, U5: footprint Connector_PinSocket_2.00mm:PinSocket_1x06_P2.00mm_Vertical -> Connector_JST:JST_SH_BM06B-SRSS-TB_1x06-1MP_P1.00mm_Vertical
- moved R6 17.4 mm to (169.7, 127.5)
- moved R2 17.4 mm to (166.6, 117.4)
- moved R4 17.3 mm to (154.7, 117.3)
- moved R8 17.3 mm to (151.6, 127.5)
- moved J2 13.5 mm to (168.1, 107.7)
- moved U1 13.5 mm to (160.3, 106.5)
- moved C10 11.8 mm to (188.8, 71.0), turned to 180 degrees
- moved SK4 11.4 mm to (160.0, 124.7)
- moved S1 9.38 mm to (198.2, 67.8), turned to 90 degrees
- moved U5 7.39 mm to (149.9, 79.0), turned to 0 degrees
- moved U4 5.54 mm to (172.2, 79.0), turned to 0 degrees
- moved C9 4.80 mm to (180.0, 72.2)
- moved T4 4.64 mm to (155.0, 60.0)
- moved C1 3.59 mm to (171.8, 59.2)
- moved C3 3.53 mm to (171.7, 65.3)
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Connections:
- J1 pad 1: Net-(J1-Pad1) -> unconnected-(J1-Pad1)
- U1 pad 15: Net-(U1-Pad15) -> unconnected-(U1-Pad15)
- U1 pad 18: Net-(U1-Pad18) -> unconnected-(U1-Pad18)
- U1 pad 19: Net-(U1-Pad19) -> unconnected-(U1-Pad19)
- U1 pad 31: Net-(U1-Pad31) -> unconnected-(U1-Pad31)
- U1 pad 32: Net-(U1-Pad32) -> unconnected-(U1-Pad32)
- U1 pad 38: Net-(U1-Pad38) -> unconnected-(U1-Pad38)
- U1 pad 41: Net-(U1-Pad41) -> unconnected-(U1-Pad41)
- U1 pad 42: Net-(U1-Pad42) -> unconnected-(U1-Pad42)
- U1 pad 43: Net-(U1-Pad43) -> unconnected-(U1-Pad43)
- U1 pad 44: Net-(U1-Pad44) -> unconnected-(U1-Pad44)
Routing:
- net /D-: track 0.00 -> 36.7 mm, vias 0 -> 1
- net /D+: track 0.00 -> 27.6 mm
- net /VUSB: track 76.9 -> 102.6 mm, vias 1 -> 2
- net /M1_encoder_B: track 68.5 -> 45.9 mm, vias 0 -> 3
- net Net-(D1-Pad1): track 7.59 -> 25.2 mm, vias 0 -> 1
- net /M2_encoder_A: track 35.1 -> 18.6 mm, vias 0 -> 1
- net /5v: track 456.9 -> 473.2 mm, vias 1 -> 3
- net /V_METER: track 70.7 -> 56.1 mm, vias 2 -> 1
- net /M2_encoder_B: track 36.1 -> 21.6 mm, vias 0 -> 1
- net Net-(R8-Pad2): track 28.6 -> 43.0 mm
- net /M1_encoder_A: track 64.9 -> 50.8 mm, vias 0 -> 1
- net /Emitter_1: track 4.24 -> 17.7 mm
- net /Emitter_3: track 4.14 -> 17.6 mm
- net /M2_speed: track 47.3 -> 33.8 mm
- net /PUSH_SW2: track 62.0 -> 48.8 mm
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Other:
- net class Default removed
- board text added: "5V |"
- board text added: "BATT"
- board text added: "GND |"
- board text added: "HC05_KEY |"
- board text added: "HC05_Key"
- board text added: "HC05_RX |"
- board text added: "J. Low, C. Diaz, T. Tang Kit-Mouse v1.2 2022"
- board text added: "Type-C (optional)"
- board text removed: "J. Low, C. Diaz Kit-Mouse v1.1 2021"
